Commit message: Update standard params.

File: urdf/standard/gimbal.urdf.xacro (robot description, xacro)
@@ -2,6 +2,6 @@
 <robot xmlns:xacro="http://www.ros.org/wiki/xacro">
     <xacro:property name="threshold" value="0.08"/>
-    <xacro:property name="pitch_lower_limit" value="-0.72"/>
-    <xacro:property name="pitch_upper_limit" value="0.457"/>
+    <xacro:property name="pitch_lower_limit" value="-0.896"/>
+    <xacro:property name="pitch_upper_limit" value="0.505"/>
     <link name="yaw">
         <inertial>

File: urdf/standard3/gimbal.transmission.urdf.xacro (robot description, xacro)
@@ -7,5 +7,5 @@
         </actuator>
         <joint name="yaw_joint">
-            <offset>-0.502</offset>
+            <offset>2.639</offset>
             <hardwareInterface>hardware_interface/EffortJointInterface</hardwareInterface>
         </joint>
@@ -17,5 +17,5 @@
         </actuator>
         <joint name="pitch_joint">
-            <offset>0.483</offset>
+            <offset>0.523</offset>
             <hardwareInterface>hardware_interface/EffortJointInterface</hardwareInterface>
         </joint>

File: urdf/standard3/standard3.urdf.xacro (robot description, xacro)
@@ -20,5 +20,5 @@
                                  camera_sim="$(arg use_simulation)"/>
             <xacro:camera_optical_frame xyz="0.06559775176285364 0.000187 0.08746327160978175"
-                                        rpy="-1.6147075 0.0527913 -1.5897212"
+                                        rpy="-1.6347075 0.0527913 -1.5897212"
                                         frame_id="$(arg camera_optical_frame)"
                                         parent="pitch"

File: urdf/standard5/gimbal.transmission.urdf.xacro (robot description, xacro)
@@ -7,5 +7,5 @@
         </actuator>
         <joint name="yaw_joint">
-            <offset>-1.5395</offset>
+            <offset>0.5436</offset>
             <hardwareInterface>hardware_interface/EffortJointInterface</hardwareInterface>
         </joint>
@@ -17,5 +17,5 @@
         </actuator>
         <joint name="pitch_joint">
-            <offset>0.415</offset>
+            <offset>0.530</offset>
             <hardwareInterface>hardware_interface/EffortJointInterface</hardwareInterface>
         </joint>

File: urdf/standard5/standard5.urdf.xacro (robot description, xacro)
@@ -20,5 +20,5 @@
                                  camera_sim="$(arg use_simulation)"/>
             <xacro:camera_optical_frame xyz="0.06559775176285364 0.000187 0.08746327160978175"
-                                        rpy="-1.6547075 0.0527913 -1.5597212"
+                                        rpy="-1.6347075 0.0527913 -1.5897212"
                                         frame_id="$(arg camera_optical_frame)"
                                         parent="pitch"
