Commit message: New balance standard.

File: urdf/balance/chassis.urdf.xacro (robot description, xacro)
@@ -1,21 +1,16 @@
 <robot xmlns:xacro="http://www.ros.org/wiki/xacro">
-    <xacro:include filename="$(find rm_description)/urdf/balance/reaction_wheel.urdf.xacro"/>
-    <xacro:include filename="$(find rm_description)/urdf/common/swerve_drive.urdf.xacro"/>
+    <xacro:include filename="$(find rm_description)/urdf/balance/momentum_block.urdf.xacro"/>
     <!-- https://upload.wikimedia.org/wikipedia/commons/5/52/Wheelbase_and_Track.png -->
-    <xacro:property name="wheel_base" value="0.328"/>
-    <xacro:property name="pivot_offset_z" value="0.12135"/>
-    <xacro:macro name="chassis">
-        <link name="base_link">
-            <inertial>
-                <mass value="6.453809"/>
-                <origin xyz="-0.013181 0.000104 0.1638"/>
-                <inertia ixx="9.725e-2" ixy="4.574e-5" ixz="7.354e-3" iyy="9.525e-2"
-                         iyz="1.021e-5" izz="1.468e-1"/>
-            </inertial>
+    <xacro:property name="wheel_base" value="0.420"/>
+    <xacro:property name="wheel_z_offset" value="0"/>
+    <xacro:property name="wheel_joint_effort" value="5"/>
+    <xacro:property name="wheel_joint_velocity" value="50"/>
+    <xacro:macro name="wheel"
+                 params="connected_to prefix wheel_x_offset wheel_y_offset wheel_z_offset  mechanical_reduction">
+        <link name="${prefix}_wheel">
             <visual>
                 <origin xyz="0 0 0" rpy="0 0 0"/>
                 <geometry>
-                    <mesh filename="package://rm_description/meshes/balance/base_link.stl"
-                          scale="0.001 .001 0.001"/>
+                    <mesh filename="package://rm_description/meshes/balance/wheel.stl" scale="0.001 .001 0.001"/>
                 </geometry>
             </visual>
@@ -23,20 +18,57 @@
                 <origin xyz="0 0 0" rpy="0 0 0"/>
                 <geometry>
-                    <mesh filename="package://rm_description/meshes/balance/base_link.stl"
-                          scale="0.001 0.001 0.001"/>
+                    <mesh filename="package://rm_description/meshes/balance/wheel.stl" scale="0.001 .001 0.001"/>
+                </geometry>
+            </collision>
+            <inertial>
+                <mass value="2.6"/>
+                <origin xyz="0 0 0"/>
+                <inertia ixx="9.115e-3" ixy="-1513.324e-9" ixz="-4566.397e-9" iyy="1.683e-2"
+                         iyz="-1.382e-4" izz="9.470e-3"/>
+            </inertial>
+        </link>
+        <joint name="${prefix}_wheel_joint" type="revolute">
+            <axis xyz="0 1 0"/>
+            <origin xyz="${wheel_x_offset} ${wheel_y_offset} ${wheel_z_offset}" rpy="0 0 0"/>
+            <parent link="${connected_to}"/>
+            <child link="${prefix}_wheel"/>
+            <limit effort="${wheel_joint_effort}" velocity="${wheel_joint_velocity}" lower="-1e16" upper="1e16"/>
+        </joint>
+        <transmission name="${prefix}_wheel_joint_trans">
+            <type>transmission_interface/SimpleTransmission</type>
+            <actuator name="${prefix}_wheel_joint_motor">
+                <mechanicalReduction>${mechanical_reduction}</mechanicalReduction>
+            </actuator>
+            <joint name="${prefix}_wheel_joint">
+                <hardwareInterface>hardware_interface/EffortJointInterface</hardwareInterface>
+            </joint>
+        </transmission>
+    </xacro:macro>
+    <xacro:macro name="chassis">
+        <link name="base_link">
+            <inertial>
+                <mass value="10.098"/>
+                <origin xyz="0.007 -0.001 0.039"/>
+                <inertia ixx="2.398e-1" ixy="-1.144e-3" ixz="3.641e-3" iyy="1.639e-1"
+                         iyz="1.525e-4" izz="3.255e-1"/>
+            </inertial>
+            <visual>
+                <origin xyz="0 0 0" rpy="0 0 0"/>
+                <geometry>
+                    <mesh filename="package://rm_description/meshes/balance/base_link.stl" scale="0.001 .001 0.001"/>
+                </geometry>
+            </visual>
+            <collision>
+                <origin xyz="0 0 0" rpy="0 0 0"/>
+                <geometry>
+                    <mesh filename="package://rm_description/meshes/balance/base_link.stl" scale="0.001 .001 0.001"/>
                 </geometry>
             </collision>
         </link>
-        <xacro:reaction_wheel connected_to="base_link"
-                              wheel_x_offset="0" wheel_y_offset="0"
-                              wheel_z_offset="0.22" mechanical_reduction="-0.166"/>
-        <xacro:swerve_drive prefix="left" connected_to="base_link"
-                            x_offset="0" y_offset="${wheel_base/2}"
-                            z_offset="${pivot_offset_z}"/>
-        <xacro:swerve_drive prefix="right" connected_to="base_link"
-                            x_offset="0" y_offset="${-wheel_base/2}"
-                            z_offset="${pivot_offset_z}"/>
-        <xacro:swerve_transmission prefix="left" wheel_reduction="13.733" pivot_offset="0"/>
-        <xacro:swerve_transmission prefix="right" wheel_reduction="-13.733" pivot_offset="1.861"/>
+        <xacro:momentum_block connected_to="base_link" block_z_offset="0.0815" mechanical_reduction="-0.166"/>
+        <xacro:wheel connected_to="base_link" prefix="left" wheel_x_offset="0" wheel_y_offset="${wheel_base/2}"
+                     wheel_z_offset="${wheel_z_offset}" mechanical_reduction="19.2032"/>
+        <xacro:wheel connected_to="base_link" prefix="right" wheel_x_offset="0" wheel_y_offset="${-wheel_base/2}"
+                     wheel_z_offset="${wheel_z_offset}" mechanical_reduction="19.2032"/>
     </xacro:macro>
 </robot>

Commit message: Change momentum block number from 1 to 2.

File: urdf/balance/chassis.urdf.xacro (robot description, xacro)
@@ -66,5 +66,10 @@
             </collision>
         </link>
-        <xacro:momentum_block connected_to="base_link" block_z_offset="0.0815" mechanical_reduction="-0.166"/>
+        <xacro:momentum_block prefix="left" reflect="1" connected_to="base_link" x_offset="0" y_offset="0.16"
+                              z_offset="0.0815"
+                              mechanical_reduction="-0.166"/>
+        <xacro:momentum_block prefix="right" reflect="-1" connected_to="base_link" x_offset="0" y_offset="-0.16"
+                              z_offset="0.0815"
+                              mechanical_reduction="-0.166"/>
         <xacro:wheel connected_to="base_link" prefix="left" wheel_x_offset="0" wheel_y_offset="${wheel_base/2}"
                      wheel_z_offset="${wheel_z_offset}" mechanical_reduction="19.2032"/>

File: urdf/balance/momentum_block.urdf.xacro (robot description, xacro)
@@ -1,12 +1,12 @@
 <robot xmlns:xacro="http://www.ros.org/wiki/xacro">
-    <xacro:property name="max_effort" value="6"/>
-    <xacro:property name="max_velocity" value="76"/>
+    <xacro:property name="max_effort" value="80"/>
+    <xacro:property name="max_velocity" value="1"/>
     <xacro:macro name="momentum_block"
-                 params="connected_to block_z_offset mechanical_reduction">
-        <link name="momentum_block">
+                 params="prefix reflect connected_to x_offset y_offset z_offset mechanical_reduction">
+        <link name="${prefix}_momentum_block">
             <visual>
                 <origin xyz="0 0 0" rpy="0 0 0"/>
                 <geometry>
-                    <mesh filename="package://rm_description/meshes/balance/momentum_block.stl"
+                    <mesh filename="package://rm_description/meshes/balance/${prefix}_momentum_block.stl"
                           scale="0.001 .001 0.001"/>
                 </geometry>
@@ -15,28 +15,35 @@
                 <origin xyz="0 0 0" rpy="0 0 0"/>
                 <geometry>
-                    <mesh filename="package://rm_description/meshes/balance/momentum_block.stl"
+                    <mesh filename="package://rm_description/meshes/balance/${prefix}_momentum_block.stl"
                           scale="0.001 .001 0.001"/>
                 </geometry>
             </collision>
             <inertial>
-                <mass value="1.854"/>
-                <origin xyz="0 0 0.0574"/>
-                <inertia ixx="4.802e-2" ixy="2046.479e-9" ixz="4753.67e-9" iyy="2.088e-3" iyz="2.759e-4"
-                         izz="4.778e-2"/>
+                <mass value="0.927"/>
+                <xacro:if value="${reflect == 1}">
+                    <origin xyz="0 -2.777e-3 45.973e-3"/>
+                    <inertia ixx="8.631E-4" ixy="3829.845E-9" ixz="1971.977E-9" iyy="9.715E-4" iyz="38124.117E-9"
+                             izz="5.924E-4"/>
+                </xacro:if>
+                <xacro:if value="${reflect == -1}">
+                    <origin xyz="0 2.777e-3 45.973e-3"/>
+                    <inertia ixx="7.732E-4" ixy="-3626.93e-9" ixz="2700.793e-9" iyy="8.723E-4" iyz="-15322.801E-9"
+                             izz="5.675E-4"/>
+                </xacro:if>
             </inertial>
         </link>
-        <joint name="momentum_block_joint" type="prismatic">
+        <joint name="${prefix}_momentum_block_joint" type="prismatic">
             <axis xyz="1 0 0"/>
-            <origin xyz="0 0 ${block_z_offset}" rpy="0 0 0"/>
+            <origin xyz="${x_offset} ${y_offset} ${z_offset}" rpy="0 0 0"/>
             <parent link="${connected_to}"/>
-            <child link="momentum_block"/>
+            <child link="${prefix}_momentum_block"/>
             <limit effort="${max_effort}" velocity="${max_velocity}" lower="-0.14" upper="0.14"/>
         </joint>
-        <transmission name="momentum_block_joint_trans">
+        <transmission name="${prefix}_momentum_block_joint_trans">
             <type>transmission_interface/SimpleTransmission</type>
-            <actuator name="momentum_block_joint_motor">
+            <actuator name="${prefix}_momentum_block_joint_motor">
                 <mechanicalReduction>${mechanical_reduction}</mechanicalReduction>
             </actuator>
-            <joint name="momentum_block_joint">
+            <joint name="${prefix}_momentum_block_joint">
                 <hardwareInterface>hardware_interface/EffortJointInterface</hardwareInterface>
             </joint>

Commit message: Update balance standard urdf.

File: urdf/balance/chassis.urdf.xacro (robot description, xacro)
@@ -68,12 +68,12 @@
         <xacro:momentum_block prefix="left" reflect="1" connected_to="base_link" x_offset="0" y_offset="0.16"
                               z_offset="0.0815"
-                              mechanical_reduction="-0.166"/>
+                              mechanical_reduction="22.22"/>
         <xacro:momentum_block prefix="right" reflect="-1" connected_to="base_link" x_offset="0" y_offset="-0.16"
                               z_offset="0.0815"
-                              mechanical_reduction="-0.166"/>
+                              mechanical_reduction="-22.22"/>
         <xacro:wheel connected_to="base_link" prefix="left" wheel_x_offset="0" wheel_y_offset="${wheel_base/2}"
                      wheel_z_offset="${wheel_z_offset}" mechanical_reduction="19.2032"/>
         <xacro:wheel connected_to="base_link" prefix="right" wheel_x_offset="0" wheel_y_offset="${-wheel_base/2}"
-                     wheel_z_offset="${wheel_z_offset}" mechanical_reduction="19.2032"/>
+                     wheel_z_offset="${wheel_z_offset}" mechanical_reduction="-19.2032"/>
     </xacro:macro>
 </robot>

File: urdf/balance/momentum_block.urdf.xacro (robot description, xacro)
@@ -1,5 +1,7 @@
 <robot xmlns:xacro="http://www.ros.org/wiki/xacro">
-    <xacro:property name="max_effort" value="80"/>
-    <xacro:property name="max_velocity" value="1"/>
+    <xacro:property name="max_effort" value="26.66"/>
+    <xacro:property name="max_velocity" value="1.395"/>
+    <xacro:property name="momentum_block_limit" value="0.14"/>
+    <xacro:property name="threshold" value="0.01"/>
     <xacro:macro name="momentum_block"
                  params="prefix reflect connected_to x_offset y_offset z_offset mechanical_reduction">
@@ -38,5 +40,9 @@
             <parent link="${connected_to}"/>
             <child link="${prefix}_momentum_block"/>
-            <limit effort="${max_effort}" velocity="${max_velocity}" lower="-0.14" upper="0.14"/>
+            <limit effort="${max_effort}" velocity="${max_velocity}" lower="${-momentum_block_limit}"
+                   upper="${momentum_block_limit}"/>
+            <safety_controller k_position="100" k_velocity="0.1"
+                               soft_lower_limit="${-momentum_block_limit+threshold}"
+                               soft_upper_limit="${momentum_block_limit-threshold}"/>
         </joint>
         <transmission name="${prefix}_momentum_block_joint_trans">
