Commit message: Adjust momentum_block limit and soft_limit.

File: urdf/balance/momentum_block.urdf.xacro (robot description, xacro)
@@ -2,6 +2,7 @@
     <xacro:property name="max_effort" value="26.66"/>
     <xacro:property name="max_velocity" value="1.395"/>
-    <xacro:property name="momentum_block_limit" value="0.14"/>
-    <xacro:property name="threshold" value="0.01"/>
+    <xacro:property name="momentum_block_upper_limit" value="0.115"/>
+    <xacro:property name="momentum_block_lower_limit" value="-0.15"/>
+    <xacro:property name="threshold" value="0.001"/>
     <xacro:macro name="momentum_block"
                  params="prefix reflect connected_to x_offset y_offset z_offset mechanical_reduction">
@@ -40,9 +41,9 @@
             <parent link="${connected_to}"/>
             <child link="${prefix}_momentum_block"/>
-            <limit effort="${max_effort}" velocity="${max_velocity}" lower="${-momentum_block_limit}"
-                   upper="${momentum_block_limit}"/>
-            <safety_controller k_position="100" k_velocity="0.1"
-                               soft_lower_limit="${-momentum_block_limit+threshold}"
-                               soft_upper_limit="${momentum_block_limit-threshold}"/>
+            <limit effort="${max_effort}" velocity="${max_velocity}" lower="${momentum_block_lower_limit}"
+                   upper="${momentum_block_upper_limit}"/>
+            <safety_controller k_position="1000" k_velocity="10"
+                               soft_lower_limit="${momentum_block_lower_limit+threshold}"
+                               soft_upper_limit="${momentum_block_upper_limit-threshold}"/>
         </joint>
         <transmission name="${prefix}_momentum_block_joint_trans">
@@ -52,4 +53,5 @@
             </actuator>
             <joint name="${prefix}_momentum_block_joint">
+                <offset>0.116</offset>
                 <hardwareInterface>hardware_interface/EffortJointInterface</hardwareInterface>
             </joint>
