Commit message: Update balance standard params.

File: urdf/balance/balance.urdf.xacro (robot description, xacro)
@@ -9,5 +9,5 @@
         <xacro:chassis/>
         <xacro:include filename="$(find rm_description)/urdf/common/imu.urdf.xacro"/>
-        <xacro:IMU connected_to="base_link" imu_name="base_imu" xyz="0.08 0. 0.08" rpy="0 0 0"/>
+        <xacro:IMU connected_to="base_link" imu_name="base_imu" xyz="0.08 0. 0.08" rpy="0 0 ${-pi/2}"/>
         <xacro:if value="$(arg load_gimbal)">
             <xacro:if value="$(arg load_shooter)">

File: urdf/balance/momentum_block.urdf.xacro (robot description, xacro)
@@ -2,7 +2,7 @@
     <xacro:property name="max_effort" value="26.66"/>
     <xacro:property name="max_velocity" value="1.395"/>
-    <xacro:property name="momentum_block_upper_limit" value="0.115"/>
-    <xacro:property name="momentum_block_lower_limit" value="-0.15"/>
-    <xacro:property name="threshold" value="0.001"/>
+    <xacro:property name="momentum_block_upper_limit" value="0.156"/>
+    <xacro:property name="momentum_block_lower_limit" value="-0.1096"/>
+    <xacro:property name="threshold" value="0.003"/>
     <xacro:macro name="momentum_block"
                  params="prefix reflect connected_to x_offset y_offset z_offset mechanical_reduction">
@@ -53,5 +53,5 @@
             </actuator>
             <joint name="${prefix}_momentum_block_joint">
-                <offset>0.116</offset>
+                <offset>0.157</offset>
                 <hardwareInterface>hardware_interface/EffortJointInterface</hardwareInterface>
             </joint>

Commit message: Complete part of urdf.

File: urdf/balance/balance.urdf.xacro (robot description, xacro)
@@ -4,4 +4,6 @@
     <xacro:arg name="load_gimbal" default="true"/>
     <xacro:arg name="load_shooter" default="true"/>
+    <xacro:arg name="camera_link" default="camera_link"/>
+    <xacro:arg name="camera_optical_frame" default="camera_optical_frame"/>
     <xacro:arg name="use_simulation" default="true"/>
     <xacro:if value="$(arg load_chassis)">
@@ -11,5 +13,21 @@
         <xacro:IMU connected_to="base_link" imu_name="base_imu" xyz="0.08 0. 0.08" rpy="0 0 ${-pi/2}"/>
         <xacro:if value="$(arg load_gimbal)">
+            <xacro:include filename="$(find rm_description)/urdf/balance/gimbal.urdf.xacro"/>
+            <xacro:include filename="$(find rm_description)/urdf/balance/gimbal.transmission.urdf.xacro"/>
+            <xacro:include filename="$(find rm_description)/urdf/common/camera.urdf.xacro"/>
+            <xacro:include filename="$(find rm_description)/urdf/common/imu.urdf.xacro"/>
+            <xacro:camera_sensor xyz="0 0 0.0887" rpy="0 0 0" frame_id="$(arg camera_link)" parent="pitch"
+                                 camera_sim="$(arg use_simulation)"/>
+            <xacro:camera_optical_frame xyz="0.06559775176285364 0.000187 0.08746327160978175"
+                                        rpy="-1.6347075 0.0527913 -1.5897212"
+                                        frame_id="$(arg camera_optical_frame)"
+                                        parent="pitch"
+                                        camera_sim="false"/>
+            <xacro:IMU connected_to="pitch" imu_name="gimbal_imu"
+                       xyz="0.00246956 0.04105199 -0.07160856"
+                       rpy="${pi} 0 ${-pi/2}"/>
             <xacro:if value="$(arg load_shooter)">
+                <xacro:include filename="$(find rm_description)/urdf/balance/shooter.urdf.xacro"/>
+                <xacro:include filename="$(find rm_description)/urdf/balance/shooter.transmission.urdf.xacro"/>
             </xacro:if>
         </xacro:if>

File: urdf/balance/chassis.urdf.xacro (robot description, xacro)
@@ -22,5 +22,5 @@
             </collision>
             <inertial>
-                <mass value="2.6"/>
+                <mass value="0.72"/>
                 <origin xyz="0 0 0"/>
                 <inertia ixx="9.115e-3" ixy="-1513.324e-9" ixz="-4566.397e-9" iyy="1.683e-2"

File: urdf/balance/gimbal.transmission.urdf.xacro (robot description, xacro)
@@ -4,8 +4,8 @@
         <type>transmission_interface/SimpleTransmission</type>
         <actuator name="yaw_joint_motor">
-            <mechanicalReduction>-1</mechanicalReduction>
+            <mechanicalReduction>1</mechanicalReduction>
         </actuator>
         <joint name="yaw_joint">
-            <offset>-0.561505488</offset>
+            <offset>-2.606</offset>
             <hardwareInterface>hardware_interface/EffortJointInterface</hardwareInterface>
         </joint>
@@ -17,5 +17,5 @@
         </actuator>
         <joint name="pitch_joint">
-            <offset>2.180819812</offset>
+            <offset>0</offset>
             <hardwareInterface>hardware_interface/EffortJointInterface</hardwareInterface>
         </joint>

File: urdf/balance/gimbal.urdf.xacro (robot description, xacro)
@@ -54,5 +54,5 @@
     </link>
     <joint name="pitch_joint" type="revolute">
-        <origin xyz="-0.05 0 0.151" rpy="0 0 0"/>
+        <origin xyz="0 0 0.151" rpy="0 0 0"/>
         <dynamics damping="0.0" friction="0.1"/>
         <limit effort="1.2" velocity="13.82" lower="${pitch_lower_limit}" upper="${pitch_upper_limit}"/>

File: urdf/balance/shooter.transmission.urdf.xacro (robot description, xacro)
@@ -4,9 +4,9 @@
         <type>transmission_interface/SimpleTransmission</type>
         <actuator name="trigger_joint_motor">
-            <mechanicalReduction>69.544</mechanicalReduction>
+            <mechanicalReduction>1</mechanicalReduction>
         </actuator>
         <joint name="trigger_joint">
             <hardwareInterface>hardware_interface/EffortJointInterface</hardwareInterface>
-            <offset>0.4</offset>
+            <offset>0.1</offset>
         </joint>
     </transmission>
@@ -29,3 +29,13 @@
         </joint>
     </transmission>
+    <transmission name="trans_cover_joint">
+        <type>transmission_interface/SimpleTransmission</type>
+        <actuator name="cover_joint_motor">
+            <mechanicalReduction>-1</mechanicalReduction>
+        </actuator>
+        <joint name="cover_joint">
+            <offset>0</offset>
+            <hardwareInterface>hardware_interface/EffortJointInterface</hardwareInterface>
+        </joint>
+    </transmission>
 </robot>

File: urdf/balance/shooter.urdf.xacro (robot description, xacro)
@@ -33,8 +33,8 @@
         <origin xyz="0 0 0.0223" rpy="0 0 0"/>
         <dynamics damping="0.0" friction="0.01"/>
-        <limit effort="18" velocity="13.5327" lower="-1e16" upper="1e16"/>
+        <limit effort="1" velocity="30" lower="-1e16" upper="1e16"/>
         <parent link="base_link"/>
         <child link="trigger"/>
-        <axis xyz="0 0 1 "/>
+        <axis xyz="0 0 1"/>
     </joint>
     <link name="cover">
